File: cad/analog/frame-control.kicad_pcb (KiCad board)
At the start: 2 copper layers, 73 parts, among them K101 LCD, K301 CONN_3, P101 JTAG, P102 TST, P103 TST, P104 TST, P105 LVDT, P106 LOADC, P201 ATX CONN, P202 TST, P203 TST, P301 TST, P302 TST, P303 TST, P304 TST, P305 TST, P306 TST, P307 BNC, P401 CONN_8X2, U101 LPC1114FBD48/302, U201 74LVCE1G06, U202 LD1117V33-DB, U301 LM4128DMF-4.1, U302 LM4040-4.1, U303 LT6011, U304 AD5662, U305 LT6011, U306 LTC1865, X101 12MHz

Commit message: added a lot more to the pcb design
Parts:
- removed C303: 100n, SM0805
- removed C304: 1u, SM0805
- added 1PIN: P***, 1pin_mech, F.Cu at (95.2, 104.4)
- added 1PIN: P***, 1pin_mech, F.Cu at (26.7, 104.4)
- added 1PIN: P***, 1pin_mech, F.Cu at (26.7, 23.1)
- added 1PIN: P***, 1pin_mech, F.Cu at (95.2, 23.1)
- added C306: 100n, SM0805, F.Cu at (52.6, 92.6)
- added C307: 100n, SM0805, F.Cu at (71.6, 84.6)
- added D202: 5VLED, LED-0805, F.Cu at (31.2, 90.4)
- added D203: 12VLED, LED-0805, F.Cu at (34.0, 90.4)
- added D204: -12VLED, LED-0805, F.Cu at (36.8, 90.4)
- added K302: COND_SIG, OSTTA030161, F.Cu at (39.4, 101.9)
- added R104: 10k, SM0805, F.Cu at (57.8, 57.4)
- added R203: 1.5k, SM0805, F.Cu at (31.2, 86.6)
- added R204: 1.5k, SM0805, F.Cu at (34.0, 86.6)
- added R205: 1.5k, SM0805, F.Cu at (36.8, 86.6)
- added R408: 10k, SM0805, F.Cu at (92.1, 26.3)
- added R409: 10k, SM0805, F.Cu at (87.6, 32.0)
- C302: value 1u -> 100n
- D201: value PWRLED -> 3v3LED
- K301: footprint PIN_ARRAY_3X1 -> OSTTA030161
- P101, P105, P106: footprint PIN_ARRAY_5x2 -> shrouded_5x2
- P401: value CONN_8X2 -> IO_PANEL; footprint pin_array_8x2 -> shrouded_8x2
- R313, R314: value 100k -> 10k
- moved D102 106.5 mm to (56.5, 26.3), turned to 90 degrees
- moved D101 104.2 mm to (54.0, 26.3), turned to 90 degrees
- moved C101 99.5 mm to (50.2, 50.4), turned to 90 degrees
- moved P201 94.4 mm to (32.0, 53.6), turned to 90 degrees
- moved R103 94.2 mm to (59.1, 22.5), turned to 90 degrees
- moved K301 93.0 mm to (66.7, 101.9)
- moved C103 91.5 mm to (52.1, 62.5), turned to 180 degrees
- moved R313 89.2 mm to (45.6, 80.5), turned to 90 degrees
- moved X101 88.7 mm to (62.2, 62.5)
- moved R201 87.9 mm to (39.6, 37.6)
- moved R102 87.7 mm to (56.5, 22.5), turned to 90 degrees
- moved C104 86.9 mm to (52.7, 50.4), turned to 90 degrees
- moved R306 85.2 mm to (55.5, 86.7)
- moved R302 84.7 mm to (51.1, 87.4)
- moved P102 83.7 mm to (54.0, 29.5)
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Connections:
- C302 pad 2: AGND -> GND
- C305 pad 2: AGND -> GND
- D101 pad 1: N-0000014 -> N-0000051
- D101 pad 2: N-0000053 -> N-0000052
- D102 pad 1: N-0000021 -> N-0000049
- D102 pad 2: N-0000052 -> N-0000050
- D103 pad 1: N-0000022 -> N-0000053
- K301 pad 2: GND -> AGND
- P102 pad 1: N-0000053 -> N-0000051
- P103 pad 1: N-0000052 -> N-0000049
- P104 pad 1: N-0000054 -> N-0000053
- P106 pad 8: N-000004 -> N-0000010
- P307 pad 2: GND -> AGND
- P401 pad 15: (no net) -> /InterfaceButtons/Aux1
- P401 pad 16: (no net) -> /InterfaceButtons/Aux2
- R101 pad 1: N-0000053 -> N-0000052
- R102 pad 1: N-0000052 -> N-0000050
- U101 pad 1: N-000004 -> (no net)
- U101 pad 14: N-0000022 -> N-0000053
- U101 pad 15: N-0000021 -> N-0000049
- U101 pad 16: N-0000014 -> N-0000051
- U101 pad 20: (no net) -> N-0000010
- U101 pad 4: (no net) -> N-0000037
- U303 pad 3: GND -> AGND
- U303 pad 5: GND -> AGND
- U305 pad 3: GND -> AGND
- U305 pad 5: GND -> AGND
Routing:
- net GND: track 0.00 -> 420.0 mm, vias 0 -> 1
- net +5V: track 0.00 -> 286.1 mm, vias 0 -> 2
- net +12V: track 0.00 -> 123.2 mm, vias 0 -> 3
- net /Analog Frontend/ADCCLK: track 0.00 -> 117.1 mm
- net -12V: track 0.00 -> 79.9 mm, vias 0 -> 3
- net N-0000069: track 0.00 -> 71.9 mm
- net /Power/PWRGD: track 0.00 -> 68.8 mm, vias 0 -> 1
- net N-0000033: track 0.00 -> 66.5 mm
- net N-0000073: track 0.00 -> 59.8 mm, vias 0 -> 1
- net N-0000049: track 0.00 -> 58.9 mm, vias 0 -> 1
- net N-0000051: track 0.00 -> 57.5 mm, vias 0 -> 1
- net +3.3V: track 0.00 -> 57.2 mm
- net N-0000034: track 0.00 -> 54.7 mm
- net N-0000029: track 0.00 -> 54.2 mm
- net N-0000035: track 0.00 -> 46.3 mm, vias 0 -> 1
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- added copper zone on B.Cu, net AGND
- added copper zone on F.Cu, net AGND
- added copper zone on B.Cu, net GND
- added copper zone on F.Cu, net GND
Other:
- board outline added: 76.2 x 88.9 mm
- net class Default: clearance 0.254 -> 0.1778
- rule trace_clearance: 0.254 -> 0.1778
- board text added: "1"
- board text added: "16"
- board text added: "A Goetz | B Kanyid | M Kulekevich"
- board text added: "GND"
- board text added: "Input"
- board text added: "JTAG"
- board text added: "LOAD FRAME CONTROLLER V1.0"
- board text added: "LOADC"
- board text added: "LOADC 7SEG"
- board text added: "LVDT"
- board text added: "LVDT 7SEG"
- board text added: "Mar 2013"
- board text added: "Output"
- board text added: "a"

Commit message: fixed issue with weird rendered blobs in gerbers
Parts:
- removed 1PIN (x4): P***, 1pin_mech
Changed lines of the file:
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@@
 (kicad_pcb (version 3) (host pcbnew "(2013-feb-26)-stable")
   (general
-    (links 209)
+    (links 205)
     (no_connects 0)
     (area 10.933641 19.228999 110.976088 108.279001)
@@
     (tracks 956)
     (zones 0)
-    (modules 87)
+    (modules 83)
     (nets 68)
   )
@@
     )
   )
-  (module 1pin_mech (layer F.Cu)
-    (at 95.25 104.394)
-    (descr "module 1 pin (ou trou mecanique de percage)")
-    (tags DEV)
-    (path 1pin_mech)
-    (fp_text reference 1PIN (at 0 -1200) (layer F.SilkS)
-      (effects (font (size 400 400) (thickness 100)))
-    )
-    (fp_text value P*** (at 0 1100) (layer F.SilkS) hide
-      (effects (font (size 400 400) (thickness 100)))
-    )
-    (fp_circle (center 0 0) (end 0 0) (layer F.SilkS) (width 0.15))
-    (pad "" thru_hole circle (at 0 0) (size 4.064 4.064) (drill 3.2512)
-      (layers *.Cu *.Mask F.SilkS)
-      (net 23 AGND)
-      (zone_connect 2)
-    )
-  )
-  (module 1pin_mech (layer F.Cu)
-    (at 26.67 104.394)
-    (descr "module 1 pin (ou trou mecanique de percage)")
-    (tags DEV)
-    (path 1pin_mech)
-    (fp_text reference 1PIN (at 0 -1200) (layer F.SilkS)
-      (effects (font (size 400 400) (thickness 100)))
-    )
-    (fp_text value P*** (at 0 1100) (layer F.SilkS) hide
-      (effects (font (size 400 400) (thickness 100)))
-    )
-    (fp_circle (center 0 0) (end 0 0) (layer F.SilkS) (width 0.15))
-    (pad "" thru_hole circle (at 0 0) (size 4.064 4.064) (drill 3.2512)
-      (layers *.Cu *.Mask F.SilkS)
-      (net 23 AGND)
-      (zone_connect 2)
-    )
-  )
-  (module 1pin_mech (layer F.Cu)
-    (at 26.67 23.114)
-    (descr "module 1 pin (ou trou mecanique de percage)")
-    (tags DEV)
-    (path 1pin_mech)
-    (fp_text reference 1PIN (at 0 -1200) (layer F.SilkS)
-      (effects (font (size 400 400) (thickness 100)))
-    )
-    (fp_text value P*** (at 0 1100) (layer F.SilkS) hide
-      (effects (font (size 400 400) (thickness 100)))
-    )
-    (fp_circle (center 0 0) (end 0 0) (layer F.SilkS) (width 0.15))
-    (pad "" thru_hole circle (at 0 0) (size 4.064 4.064) (drill 3.2512)
-      (layers *.Cu *.Mask F.SilkS)
-      (net 24 GND)
-      (zone_connect 2)
-    )
-  )
-  (module 1pin_mech (layer F.Cu)
-    (at 95.25 23.114)
-    (descr "module 1 pin (ou trou mecanique de percage)")
-    (tags DEV)
-    (path 1pin_mech)
-    (fp_text reference 1PIN (at 0 -1200) (layer F.SilkS)
-      (effects (font (size 400 400) (thickness 100)))
-    )
-    (fp_text value P*** (at 0 1100) (layer F.SilkS) hide
-      (effects (font (size 400 400) (thickness 100)))
-    )
-    (fp_circle (center 0 0) (end 0 0) (layer F.SilkS) (width 0.15))
-    (pad "" thru_hole circle (at 0 0) (size 4.064 4.064) (drill 3.2512)
-      (layers *.Cu *.Mask F.SilkS)
-      (net 24 GND)
-      (zone_connect 2)
-    )
-  )
